File: Kicad/alarm/alarm/alarm.kicad_pcb (KiCad board)
At the start: 2 copper layers, 33 parts, among them J1 Conn_01x05_Male, J10 Conn_01x01_Male, J11 Conn_01x01_Male, J12 Conn_01x01_Male, J2 Conn_01x02_Male, J3 Conn_01x05_Male, J4 Conn_01x05_Male, J5 Conn_01x05_Male, J6 Conn_01x05_Male, J7 Conn_01x05_Male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

Commit message: q
Parts:
- added J13: Conn_01x02, footprints otg:1x02, F.Cu at (233.7, 47.5)
- added J14: Conn_01x02, footprints otg:1x02, F.Cu at (233.5, 97.5)
- added J15: Conn_01x02, footprints otg:1x02, F.Cu at (233.5, 72.5)
- R9: moved to F.Cu
- moved U1 205.4 mm to (255.5, 74.5), turned to 180 degrees
- moved R1 199.6 mm to (263.5, 74.5), turned to 0 degrees
- moved J12 198.4 mm to (231.7, 42.0)
- moved C7 194.5 mm to (237.8, 100.5)
- moved J11 194.2 mm to (227.7, 34.0)
- moved J8 193.2 mm to (231.7, 34.0)
- moved R9 191.0 mm to (234.7, 42.0), turned to -90 degrees
- moved R3 190.3 mm to (260.5, 76.5)
- moved U2 189.7 mm to (237.9, 84.5)
- moved J10 189.6 mm to (227.7, 42.0)
- moved J3 188.9 mm to (268.5, 84.5)
- moved R8 183.9 mm to (229.7, 46.0), turned to -90 degrees
- moved J1 181.9 mm to (250.5, 84.5)
- moved C9 173.8 mm to (237.8, 96.5), turned to 0 degrees
- moved R4 140.8 mm to (263.7, 49.4)
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Routing:
- net Earth: track 0.00 -> 207.9 mm
- net +3.3V: track 0.00 -> 153.6 mm
- net +5V: track 0.00 -> 134.8 mm
- net CSN2: track 0.00 -> 49.4 mm
- net CSN3: track 0.00 -> 49.3 mm
- net CSN1: track 0.00 -> 49.3 mm
- net MOSI2: track 0.00 -> 47.0 mm
- net MOSI3: track 0.00 -> 47.0 mm
- net MOSI1: track 0.00 -> 47.0 mm
- net MISO2: track 0.00 -> 43.9 mm
- net MISO3: track 0.00 -> 43.8 mm
- net MISO1: track 0.00 -> 43.8 mm
- net INPUT1: track 0.00 -> 17.1 mm
- net INPUT3: track 0.00 -> 15.1 mm
- net INPUT2: track 0.00 -> 13.8 mm
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
Commit message: a
Parts:
- J10, J11, J12, J8: footprint Connector_PinHeader_1.00mm:PinHeader_1x01_P1.00mm_Vertical -> Connector_PinHeader_2.54mm:PinHeader_1x01_P2.54mm_Vertical
- moved J10 15.4 mm to (228.6, 26.6)
- moved J8 7.40 mm to (231.7, 26.6)
- moved C3 6.40 mm to (237.9, 44.0)
- moved J13 6.40 mm to (233.7, 41.1)
- moved R4 6.40 mm to (263.7, 43.0)
- moved R9 6.40 mm to (234.7, 35.6)
- moved U3 6.40 mm to (255.8, 42.9)
- moved J7 6.40 mm to (250.7, 27.9)
- moved J9 6.40 mm to (268.7, 27.9)
- moved U6 6.40 mm to (238.1, 27.9)
- moved C4 6.40 mm to (237.9, 40.0)
- moved R5 6.40 mm to (260.7, 45.0)
- moved R8 5.40 mm to (229.7, 40.6)
- moved J12 4.40 mm to (231.7, 37.6)
- moved J11 3.71 mm to (228.6, 37.6)
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Routing:
- net +5V: track 134.8 -> 153.5 mm
- net Earth: track 207.9 -> 221.7 mm
- net Net-(J10-Pin_1): track 4.83 -> 15.2 mm
- net Net-(U5-ADJ): track 8.45 -> 5.32 mm
- net MISO1: track 43.8 -> 46.3 mm
- net MISO2: track 43.9 -> 46.3 mm
- net MISO3: track 43.8 -> 46.1 mm
- net MOSI2: track 47.0 -> 49.2 mm
- net CSN2: track 49.4 -> 51.4 mm
- net +3.3V: track 153.6 -> 155.5 mm
- net CSN3: track 49.3 -> 51.0 mm
- net CSN1: track 49.3 -> 50.8 mm
- net INPUT2: track 13.8 -> 14.8 mm
- net MOSI1: track 47.0 -> 48.0 mm
- net INPUT3: track 15.1 -> 16.1 mm
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- added copper zone on B.Cu, net Earth
