File: Kicad/alarm/alarm/alarm.kicad_sch (KiCad schematic)
At the start: 33 parts, among them J1 Conn_01x05_Male, J10 Conn_01x01_Male, J11 Conn_01x01_Male, J12 Conn_01x01_Male, J2 Conn_01x02_Male, J3 Conn_01x05_Male, J4 Conn_01x05_Male, J5 Conn_01x05_Male, J6 Conn_01x05_Male, J7 Conn_01x05_Male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

Commit message: q
Parts:
- added J13, J14, J15: Conn_01x02, footprints otg:1x02, symbol 00-OTG-Connectorer:Conn_01x02
Connections:
- net +5V: now also J13.2 (Pin_2), J14.2 (Pin_2), J15.2 (Pin_2)
- net Earth: now also J13.1 (Pin_1), J14.1 (Pin_1), J15.1 (Pin_1)

Commit message: a
Parts:
- J10, J11, J12, J8: footprint Connector_PinHeader_1.00mm:PinHeader_1x01_P1.00mm_Vertical -> Connector_PinHeader_2.54mm:PinHeader_1x01_P2.54mm_Vertical
Changed lines of the file:
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@@
       (effects (font (size 1.27 1.27)))
     )
-    (property "Footprint" "Connector_PinHeader_1.00mm:PinHeader_1x01_P1.00mm_Vertical" (at 200.66 123.19 0)
+    (property "Footprint" "Connector_PinHeader_2.54mm:PinHeader_1x01_P2.54mm_Vertical" (at 200.66 123.19 0)
       (effects (font (size 1.27 1.27)) hide)
     )
@@
       (effects (font (size 1.27 1.27)))
     )
-    (property "Footprint" "Connector_PinHeader_1.00mm:PinHeader_1x01_P1.00mm_Vertical" (at 200.66 130.81 0)
+    (property "Footprint" "Connector_PinHeader_2.54mm:PinHeader_1x01_P2.54mm_Vertical" (at 200.66 130.81 0)
       (effects (font (size 1.27 1.27)) hide)
     )
@@
       (effects (font (size 1.27 1.27)))
     )
-    (property "Footprint" "Connector_PinHeader_1.00mm:PinHeader_1x01_P1.00mm_Vertical" (at 175.26 130.81 0)
+    (property "Footprint" "Connector_PinHeader_2.54mm:PinHeader_1x01_P2.54mm_Vertical" (at 175.26 130.81 0)
       (effects (font (size 1.27 1.27)) hide)
     )
@@
       (effects (font (size 1.27 1.27)))
     )
-    (property "Footprint" "Connector_PinHeader_1.00mm:PinHeader_1x01_P1.00mm_Vertical" (at 175.26 123.19 0)
-      (effects (font (size 1.27 1.27)) hide)
-    )
+    (property "Footprint" "Connector_PinHeader_2.54mm:PinHeader_1x01_P2.54mm_Vertical" (at 175.26 123.19 0)
+      (effects (font (size 1.27 1.27)) hide)
+    )
